File: _saved_Switch Matrix.sch (KiCad schematic (older format))
At the start: 183 parts

Commit message: 2
Parts:
- D_,: renamed from D?; value D_, -> D
- D_.: renamed from D?; value D_. -> D
- D_/: renamed from D?; value D_/ -> D
- D_B: renamed from D?; value D_B -> D
- D_C: renamed from D?; value D_C -> D
- D_M: renamed from D?; value D_M -> D
- D_N: renamed from D?; value D_N -> D
- D_V: renamed from D?; value D_V -> D
- D_X: renamed from D?; value D_X -> D
- D_Z: renamed from D?; value D_Z -> D
- gave numbers to parts that had none: 19
Changed lines of the file:
@@
 $EndComp
 $Comp
-L Device:R_Small R?
+L Device:R_Small R43
 U 1 1 5D90BB18
 P 1850 3850
-F 0 "R?" H 1909 3896 50  0000 L CNN
+F 0 "R43" H 1909 3896 50  0000 L CNN
 F 1 "470" H 1909 3805 50  0000 L CNN
 F 2 "" H 1850 3850 50  0001 C CNN
@@
 $EndComp
 $Comp
-L Device:R_Small R?
+L Device:R_Small R44
 U 1 1 5D90BB27
 P 2425 3850
-F 0 "R?" H 2484 3896 50  0000 L CNN
+F 0 "R44" H 2484 3896 50  0000 L CNN
 F 1 "470" H 2484 3805 50  0000 L CNN
 F 2 "" H 2425 3850 50  0001 C CNN
@@
 $EndComp
 $Comp
-L Device:R_Small R?
+L Device:R_Small R45
 U 1 1 5D90BB36
 P 3025 3850
-F 0 "R?" H 3084 3896 50  0000 L CNN
+F 0 "R45" H 3084 3896 50  0000 L CNN
 F 1 "470" H 3084 3805 50  0000 L CNN
 F 2 "" H 3025 3850 50  0001 C CNN
@@
 $EndComp
 $Comp
-L Device:R_Small R?
+L Device:R_Small R46
 U 1 1 5D90BB45
 P 3600 3850
-F 0 "R?" H 3659 3896 50  0000 L CNN
+F 0 "R46" H 3659 3896 50  0000 L CNN
 F 1 "470" H 3659 3805 50  0000 L CNN
 F 2 "" H 3600 3850 50  0001 C CNN
@@
 $EndComp
 $Comp
-L Device:R_Small R?
+L Device:R_Small R47
 U 1 1 5D90BB54
 P 4175 3850
-F 0 "R?" H 4234 3896 50  0000 L CNN
+F 0 "R47" H 4234 3896 50  0000 L CNN
 F 1 "470" H 4234 3805 50  0000 L CNN
 F 2 "" H 4175 3850 50  0001 C CNN
@@
 $EndComp
 $Comp
-L Device:R_Small R?
+L Device:R_Small R48
 U 1 1 5D90BB63
 P 4800 3850
-F 0 "R?" H 4859 3896 50  0000 L CNN
+F 0 "R48" H 4859 3896 50  0000 L CNN
 F 1 "470" H 4859 3805 50  0000 L CNN
 F 2 "" H 4800 3850 50  0001 C CNN
@@
 $EndComp
 $Comp
-L Device:R_Small R?
+L Device:R_Small R49
 U 1 1 5D90BB72
 P 5375 3850
-F 0 "R?" H 5434 3896 50  0000 L CNN
+F 0 "R49" H 5434 3896 50  0000 L CNN
 F 1 "470" H 5434 3805 50  0000 L CNN
 F 2 "" H 5375 3850 50  0001 C CNN
@@
 $EndComp
 $Comp
-L Device:R_Small R?
+L Device:R_Small R50
 U 1 1 5D90BB81
 P 5950 3850
-F 0 "R?" H 6009 3896 50  0000 L CNN
+F 0 "R50" H 6009 3896 50  0000 L CNN
 F 1 "470" H 6009 3805 50  0000 L CNN
 F 2 "" H 5950 3850 50  0001 C CNN
@@
 $EndComp
 $Comp
-L Device:R_Small R?
+L Device:R_Small R51
 U 1 1 5D90BB90
 P 6550 3850
-F 0 "R?" H 6609 3896 50  0000 L CNN
+F 0 "R51" H 6609 3896 50  0000 L CNN
 F 1 "470" H 6609 3805 50  0000 L CNN
 F 2 "" H 6550 3850 50  0001 C CNN
@@
 $EndComp
 $Comp
-L Device:R_Small R?
+L Device:R_Small R52
 U 1 1 5D90BB9F
 P 7125 3850
-F 0 "R?" H 7184 3896 50  0000 L CNN
+F 0 "R52" H 7184 3896 50  0000 L CNN
 F 1 "470" H 7184 3805 50  0000 L CNN
 F 2 "" H 7125 3850 50  0001 C CNN
@@
 $EndComp
 $Comp
-L Device:R_Small R?
+L Device:R_Small R53
 U 1 1 5D90BBAE
 P 7700 3850
-F 0 "R?" H 7759 3896 50  0000 L CNN
+F 0 "R53" H 7759 3896 50  0000 L CNN
 F 1 "470" H 7759 3805 50  0000 L CNN
 F 2 "" H 7700 3850 50  0001 C CNN
@@
 $EndComp
 $Comp
-L Device:R_Small R?
+L Device:R_Small R54
 U 1 1 5D90BBDB
 P 1275 4600
-F 0 "R?" H 1334 4646 50  0000 L CNN
+F 0 "R54" H 1334 4646 50  0000 L CNN
 F 1 "470" H 1334 4555 50  0000 L CNN
 F 2 "" H 1275 4600 50  0001 C CNN
@@
 $EndComp
 $Comp
-L Device:R_Small R?
+L Device:R_Small R55
 U 1 1 5D90BBEA
 P 1850 4600
-F 0 "R?" H 1909 4646 50  0000 L CNN
+F 0 "R55" H 1909 4646 50  0000 L CNN
 F 1 "470" H 1909 4555 50  0000 L CNN
 F 2 "" H 1850 4600 50  0001 C CNN
@@
 $EndComp
 $Comp
-L Device:R_Small R?
+L Device:R_Small R56
 U 1 1 5D90BBF9
 P 2425 4600
-F 0 "R?" H 2484 4646 50  0000 L CNN
+F 0 "R56" H 2484 4646 50  0000 L CNN
 F 1 "470" H 2484 4555 50  0000 L CNN
 F 2 "" H 2425 4600 50  0001 C CNN
@@
 $EndComp
 $Comp
-L Device:R_Small R?
+L Device:R_Small R57
 U 1 1 5D90BC08
 P 3025 4600
-F 0 "R?" H 3084 4646 50  0000 L CNN
+F 0 "R57" H 3084 4646 50  0000 L CNN
 F 1 "470" H 3084 4555 50  0000 L CNN
 F 2 "" H 3025 4600 50  0001 C CNN
@@
 $EndComp
 $Comp
-L Device:R_Small R?
+L Device:R_Small R58
 U 1 1 5D90BC17
 P 3600 4600
-F 0 "R?" H 3659 4646 50  0000 L CNN
+F 0 "R58" H 3659 4646 50  0000 L CNN
 F 1 "470" H 3659 4555 50  0000 L CNN
 F 2 "" H 3600 4600 50  0001 C CNN
@@
 $EndComp
 $Comp
-L Device:R_Small R?
+L Device:R_Small R59
 U 1 1 5D90BC26
 P 4175 4600
-F 0 "R?" H 4234 4646 50  0000 L CNN
+F 0 "R59" H 4234 4646 50  0000 L CNN
 F 1 "470" H 4234 4555 50  0000 L CNN
 F 2 "" H 4175 4600 50  0001 C CNN
@@
 $EndComp
 $Comp
-L Device:R_Small R?
+L Device:R_Small R60
 U 1 1 5D90BC35
 P 4800 4600
-F 0 "R?" H 4859 4646 50  0000 L CNN
+F 0 "R60" H 4859 4646 50  0000 L CNN
 F 1 "470" H 4859 4555 50  0000 L CNN
 F 2 "" H 4800 4600 50  0001 C CNN
@@
 $EndComp
 $Comp
-L Device:R_Small R?
+L Device:R_Small R61
 U 1 1 5D90BC44
 P 5375 4600
-F 0 "R?" H 5434 4646 50  0000 L CNN
+F 0 "R61" H 5434 4646 50  0000 L CNN
 F 1 "470" H 5434 4555 50  0000 L CNN
 F 2 "" H 5375 4600 50  0001 C CNN
@@
 $EndComp
 $Comp
-L Device:D_Small D?
+L Device:D_Small D_Z
 U 1 1 5D945BA6
 P 1700 3975
-F 0 "D?" V 1746 3907 50  0000 R CNN
-F 1 "D_Z" V 1655 3907 50  0000 R CNN
+F 0 "D_Z" V 1746 3907 50  0000 R CNN
+F 1 "D" V 1655 3907 50  0000 R CNN
 F 2 "" V 1700 3975 50  0001 C CNN
 F 3 "~" V 1700 3975 50  0001 C CNN
@@
 $EndComp
 $Comp
-L Device:D_Small D?
+L Device:D_Small D_X
 U 1 1 5D945BAD
 P 2275 3975
-F 0 "D?" V 2321 3907 50  0000 R CNN
-F 1 "D_X" V 2230 3907 50  0000 R CNN
+F 0 "D_X" V 2321 3907 50  0000 R CNN
+F 1 "D" V 2230 3907 50  0000 R CNN
 F 2 "" V 2275 3975 50  0001 C CNN
 F 3 "~" V 2275 3975 50  0001 C CNN
@@
 $EndComp
 $Comp
-L Device:D_Small D?
+L Device:D_Small D_C
 U 1 1 5D945BB4
 P 2875 3975
-F 0 "D?" V 2921 3907 50  0000 R CNN
-F 1 "D_C" V 2830 3907 50  0000 R CNN
+F 0 "D_C" V 2921 3907 50  0000 R CNN
+F 1 "D" V 2830 3907 50  0000 R CNN
 F 2 "" V 2875 3975 50  0001 C CNN
 F 3 "~" V 2875 3975 50  0001 C CNN
@@
 $EndComp
 $Comp
-L Device:D_Small D?
+L Device:D_Small D_V
 U 1 1 5D945BBB
 P 3450 3975
-F 0 "D?" V 3496 3907 50  0000 R CNN
-F 1 "D_V" V 3405 3907 50  0000 R CNN
+F 0 "D_V" V 3496 3907 50  0000 R CNN
+F 1 "D" V 3405 3907 50  0000 R CNN
 F 2 "" V 3450 3975 50  0001 C CNN
 F 3 "~" V 3450 3975 50  0001 C CNN
@@
 $EndComp
 $Comp
-L Device:D_Small D?
+L Device:D_Small D_B
 U 1 1 5D945BC2
 P 4025 3975
-F 0 "D?" V 4071 3907 50  0000 R CNN
-F 1 "D_B" V 3980 3907 50  0000 R CNN
+F 0 "D_B" V 4071 3907 50  0000 R CNN
+F 1 "D" V 3980 3907 50  0000 R CNN
 F 2 "" V 4025 3975 50  0001 C CNN
 F 3 "~" V 4025 3975 50  0001 C CNN
@@
 $EndComp
 $Comp
-L Device:D_Small D?
+L Device:D_Small D_N
 U 1 1 5D945BC9
 P 4650 3975
-F 0 "D?" V 4696 3907 50  0000 R CNN
-F 1 "D_N" V 4605 3907 50  0000 R CNN
+F 0 "D_N" V 4696 3907 50  0000 R CNN
+F 1 "D" V 4605 3907 50  0000 R CNN
 F 2 "" V 4650 3975 50  0001 C CNN
 F 3 "~" V 4650 3975 50  0001 C CNN
@@
 $EndComp
 $Comp
-L Device:D_Small D?
+L Device:D_Small D_M
 U 1 1 5D945BD0
 P 5225 3975
-F 0 "D?" V 5271 3907 50  0000 R CNN
-F 1 "D_M" V 5180 3907 50  0000 R CNN
+F 0 "D_M" V 5271 3907 50  0000 R CNN
+F 1 "D" V 5180 3907 50  0000 R CNN
 F 2 "" V 5225 3975 50  0001 C CNN
 F 3 "~" V 5225 3975 50  0001 C CNN
@@
 $EndComp
 $Comp
-L Device:D_Small D?
+L Device:D_Small D_,
 U 1 1 5D945BD7
 P 5800 3975
-F 0 "D?" V 5846 3907 50  0000 R CNN
-F 1 "D_," V 5755 3907 50  0000 R CNN
+F 0 "D_," V 5846 3907 50  0000 R CNN
+F 1 "D" V 5755 3907 50  0000 R CNN
 F 2 "" V 5800 3975 50  0001 C CNN
 F 3 "~" V 5800 3975 50  0001 C CNN
@@
 $EndComp
 $Comp
-L Device:D_Small D?
+L Device:D_Small D_.
 U 1 1 5D945BDE
 P 6400 3975
-F 0 "D?" V 6446 3907 50  0000 R CNN
-F 1 "D_." V 6355 3907 50  0000 R CNN
+F 0 "D_." V 6446 3907 50  0000 R CNN
+F 1 "D" V 6355 3907 50  0000 R CNN
 F 2 "" V 6400 3975 50  0001 C CNN
 F 3 "~" V 6400 3975 50  0001 C CNN
@@
 $EndComp
 $Comp
-L Device:D_Small D?
+L Device:D_Small D_/
 U 1 1 5D945BE5
 P 6975 3975
-F 0 "D?" V 7021 3907 50  0000 R CNN
-F 1 "D_/" V 6930 3907 50  0000 R CNN
+F 0 "D_/" V 7021 3907 50  0000 R CNN
+F 1 "D" V 6930 3907 50  0000 R CNN
 F 2 "" V 6975 3975 50  0001 C CNN
 F 3 "~" V 6975 3975 50  0001 C CNN
